Commit message: Added a simulated standalone version

File: urdf/hector_multisensor_head_standalone.urdf.xacro (robot description, xacro)
@@ -1,18 +1,30 @@
 <?xml version="1.0" ?>
 <robot xmlns:xacro="http://ros.org/wiki/xacro" name="hector_multisensor_head">
-  <xacro:include filename="$(find thor_mang_description)/urdf/helper_macros.urdf.xacro.xml" />
+  <!--<xacro:include filename="$(find thor_mang_description)/urdf/helper_macros.urdf.xacro.xml" />-->
   <xacro:include filename="$(find hector_components_description)/urdf/hector_multisensor_head.urdf.xacro" />
-<link name="world"/>
+  <link name="base" >
+    <visual>
+      <geometry>
+            <cylinder length="1.0" radius="0.047"/>
+      </geometry>
+    </visual>
+     <collision>
+      <geometry>
+            <cylinder length="1.0" radius="0.047"/>
+      </geometry>
+    </collision>
+  </link>
   <joint name="fixed" type="fixed">
-    <parent link="world"/>
+    <parent link="base"/>
     <child link="head_link"/>
+      <origin xyz="0.0 0.0 0.5" rpy="0 0 0"/>
   </joint>
-    <hector_multisensor_head_macro parent="world"  name="head" scaling="0.001">
-      <origin xyz="0.0 0.0 -0.006" rpy="${M_PI*0.5} ${0 } ${M_PI*0.5}"/>
+    <hector_multisensor_head_macro parent="base"  name="head" scaling="0.001">
+      <origin xyz="0.0 0.0 0" rpy="${M_PI*0.5} ${0 } ${M_PI*0.5}"/>
     </hector_multisensor_head_macro>
-      <gazebo>
+   <gazebo>
     <plugin name="gazebo_ros_control" filename="libgazebo_ros_control.so">
       <robotNamespace>thor_mang</robotNamespace>
     </plugin>
-  </gazebo>
+    </gazebo>
 </robot>

Commit message: Fixed the mount of the head

File: urdf/hector_multisensor_head_standalone.urdf.xacro (robot description, xacro)
@@ -3,17 +3,24 @@
   <!--<xacro:include filename="$(find thor_mang_description)/urdf/helper_macros.urdf.xacro.xml" />-->
   <xacro:include filename="$(find hector_components_description)/urdf/hector_multisensor_head.urdf.xacro" />
+  <link name="world"/>
+  <joint name="fixed1" type="fixed">
+    <parent link="world"/>
+    <child link="base"/>
+      <origin xyz="0.0 0.0 0.5" rpy="0 0 0"/>
+  </joint>
   <link name="base" >
+    <origin xyz="0.0 0.0 0.0" rpy="0 0 0"/>
     <visual>
       <geometry>
-            <cylinder length="1.0" radius="0.047"/>
+            <cylinder length="1" radius="0.045"/>
       </geometry>
     </visual>
      <collision>
       <geometry>
-            <cylinder length="1.0" radius="0.047"/>
+            <cylinder length="1" radius="0.045"/>
       </geometry>
     </collision>
   </link>
-  <joint name="fixed" type="fixed">
+  <joint name="fixed2" type="fixed">
     <parent link="base"/>
     <child link="head_link"/>

Commit message: Added calibration macro

File: urdf/hector_multisensor_head_standalone.urdf.xacro (robot description, xacro)
@@ -28,5 +28,8 @@
   </joint>
     <hector_multisensor_head_macro parent="base"  name="head" scaling="0.001">
-      <origin xyz="0.0 0.0 0" rpy="${M_PI*0.5} ${0 } ${M_PI*0.5}"/>
+      <origin xyz="0.0 0.0 0" rpy="${M_PI*0.5} 0 ${M_PI*0.5}"/>
+      <!-- Calibrated origin -->
+      <!--<origin xyz="0.0 4.16332e-05 0.0126342" rpy="0 0.0209768 -0.00322112"/> -->
+      <origin xyz="0.0 0.0 0.0" rpy="0 0.0 0.0"/>
     </hector_multisensor_head_macro>
    <gazebo>

Commit message: Added calibration to URDF model and improved LIDAR settings

File: urdf/hector_multisensor_head_standalone.urdf.xacro (robot description, xacro)
@@ -30,6 +30,5 @@
       <origin xyz="0.0 0.0 0" rpy="${M_PI*0.5} 0 ${M_PI*0.5}"/>
       <!-- Calibrated origin -->
-      <!--<origin xyz="0.0 4.16332e-05 0.0126342" rpy="0 0.0209768 -0.00322112"/> -->
-      <origin xyz="0.0 0.0 0.0" rpy="0 0.0 0.0"/>
+      <origin xyz="0 0.000323461 0.0127965" rpy="0 0.021197 -0.00357142"/>
     </hector_multisensor_head_macro>
    <gazebo>

Commit message: added optenv so lidar calibration is only used for the real robot

File: urdf/hector_multisensor_head_standalone.urdf.xacro (robot description, xacro)
@@ -1,5 +1,4 @@
 <?xml version="1.0" ?>
 <robot xmlns:xacro="http://ros.org/wiki/xacro" name="hector_multisensor_head">
-  <!--<xacro:include filename="$(find thor_mang_description)/urdf/helper_macros.urdf.xacro.xml" />-->
   <xacro:include filename="$(find hector_components_description)/urdf/hector_multisensor_head.urdf.xacro" />
   <link name="world"/>
@@ -7,5 +6,5 @@
     <parent link="world"/>
     <child link="base"/>
-      <origin xyz="0.0 0.0 0.5" rpy="0 0 0"/>
+    <origin xyz="0.0 0.0 0.5" rpy="0 0 0"/>
   </joint>
   <link name="base" >
@@ -25,15 +24,20 @@
     <parent link="base"/>
     <child link="head_link"/>
-      <origin xyz="0.0 0.0 0.5" rpy="0 0 0"/>
+    <origin xyz="0.0 0.0 0.5" rpy="0 0 0"/>
   </joint>
-    <hector_multisensor_head_macro parent="base"  name="head" scaling="0.001">
-      <origin xyz="0.0 0.0 0" rpy="${M_PI*0.5} 0 ${M_PI*0.5}"/>
-      <!-- Calibrated origin -->
-      <origin xyz="0 0.000323461 0.0127965" rpy="0 0.021197 -0.00357142"/>
-    </hector_multisensor_head_macro>
-   <gazebo>
-    <plugin name="gazebo_ros_control" filename="libgazebo_ros_control.so">
-      <robotNamespace>thor_mang</robotNamespace>
-    </plugin>
+  <hector_multisensor_head_macro parent="base"  name="head" scaling="0.001">
+    <origin xyz="0.0 0.0 0" rpy="${M_PI*0.5} 0 ${M_PI*0.5}"/>
+    <!-- Calibrated origin -->
+    <xacro:if value="$(optenv THOR_REAL_ROBOT false)">
+      <xacro:include filename="$(find thor_mang_description)/head_lidar_calibration/calibration.urdf.xacro" />
+    </xacro:if>
+    <xacro:unless value="$(optenv THOR_REAL_ROBOT false)">
+      <xacro:include filename="$(find thor_mang_description)/head_lidar_calibration/zero_calibration.urdf.xacro" />
+    </xacro:unless>
+  </hector_multisensor_head_macro>
+    <gazebo>
+      <plugin name="gazebo_ros_control" filename="libgazebo_ros_control.so">
+        <robotNamespace>thor_mang</robotNamespace>
+      </plugin>
     </gazebo>
 </robot>
